File: Hardware/PendulumController/PendulumController.kicad_pcb (KiCad board)
At the start: 2 copper layers, 157 x 47 mm, 67 parts, among them J101 MOTOR, J102 ENCODER, J201 ICSP, J302 19V Input, J401 USBC, J402 PROG, Q101 MMBT3904, Q102 MMBT3906, SW201 RESET, SW202 START_SW, SW203 STOP/MODE_SW, U201 ATmega328P, U301 NCV1117ST50T3G, U401 FT232RL, Y201 16mHz

Commit message: Circuiting
Parts:
- moved D301 14.0 mm to (201.0, 95.5)
- moved R301 14.0 mm to (197.0, 95.5)
- moved C101 2.00 mm to (174.0, 106.0)
- moved C401 1.00 mm to (211.0, 74.0)
- moved C402 1.00 mm to (207.5, 74.0)
- moved R208 0.06 mm to (91.6, 84.2)
- moved SW203 0.06 mm to (94.8, 81.8)
Routing:
- net +5V: track 8.24 -> 133.3 mm, vias 0 -> 2
- net +19V: track 0.00 -> 67.4 mm
- net Net-(R404-Pad2): track 0.00 -> 21.6 mm
- net Net-(A101-Pad6): track 0.00 -> 20.2 mm
- net Net-(R403-Pad1): track 0.00 -> 17.7 mm
- net Net-(A101-Pad5): track 0.00 -> 16.0 mm
- net Net-(R401-Pad1): track 0.00 -> 13.8 mm, vias 0 -> 2
- net VBUS: track 0.00 -> 13.6 mm, vias 0 -> 2
- net Net-(A101-Pad4): track 0.00 -> 11.9 mm
- net GND: track 0.00 -> 11.4 mm
- net Net-(J401-PadB5): track 0.00 -> 10.9 mm
- net Net-(J401-PadA5): track 0.00 -> 7.80 mm
- net Net-(A101-Pad3): track 0.00 -> 7.74 mm
- net /EN: track 0.00 -> 3.70 mm
- net Net-(A101-Pad13): track 0.00 -> 3.54 mm
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
Commit message: Small layout improvements
Parts:
- moved R207 5.46 mm to (107.2, 82.5)
- moved SW202 5.25 mm to (110.4, 81.8)
Connections:
- D201 pad 2: /MCU/SCK -> /MCU/STAT_LED
- U201 pad 14: unconnected-(U201-Pad14) -> /MCU/STAT_LED
Routing:
- net +5V: track 133.3 -> 226.6 mm, vias 2 -> 3
- net /EN: track 3.70 -> 14.3 mm
- net /MCU/STOP/MODE: track 0.00 -> 8.61 mm, vias 0 -> 1
- net /MCU/START: track 0.00 -> 7.12 mm, vias 0 -> 1
- net /TFT_LED: track 0.00 -> 4.79 mm
- net Net-(Q101-Pad3): track 0.00 -> 3.22 mm
- net Net-(Q102-Pad3): track 0.00 -> 2.60 mm
- net Net-(Q101-Pad1): track 0.00 -> 2.26 mm
- net Net-(Q102-Pad1): track 0.00 -> 2.17 mm
- net GND: track 11.4 -> 13.0 mm, vias 0 -> 1
Changed lines of the file:
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@@
   (net 61 "/STEP")
   (net 62 "/DIR")
-  (net 63 "unconnected-(U201-Pad14)")
+  (net 63 "/MCU/STAT_LED")
   (net 64 "/MCU/AnalogP")
   (net 65 "/MCU/AnalogI")
@@
   )
   (footprint "Resistor_SMD:R_0805_2012Metric" (layer "F.Cu")
-    (at 112.5 84)
+    (at 107.25 82.5)
     (descr "Resistor SMD 0805 (2012 Metric), square (rectangular) end terminal, IPC_7351 nominal, (Body size source: IPC-SM-782 page 72, https://www.pcb-3d.com/wordpress/wp-content/uploads/ipc-sm-782a_amendment_1_and_2.pdf), generated with kicad-footprint-generator")
     (tags "resistor")
@@
       (net 6 "Net-(D201-Pad1)") (pinfunction "K") (pintype "passive"))
     (pad "2" smd roundrect (at 0.9375 0 90) (size 0.975 1.4) (layers "F.Cu" "F.Paste" "F.Mask") (roundrect_rratio 0.25)
-      (net 68 "/MCU/SCK") (pinfunction "A") (pintype "passive"))
+      (net 63 "/MCU/STAT_LED") (pinfunction "A") (pintype "passive"))
     (model "${KICAD6_3DMODEL_DIR}/LED_SMD.3dshapes/LED_0805_2012Metric.wrl"
       (offset (xyz 0 0 0))
@@
       (net 20 "/MCU/START") (pinfunction "PB1") (pintype "bidirectional"))
     (pad "14" smd rect (at 1.2 4.25 135) (size 1.6 0.55) (layers "F.Cu" "F.Paste" "F.Mask")
-      (net 63 "unconnected-(U201-Pad14)") (pinfunction "PB2") (pintype "bidirectional+no_connect"))
+      (net 63 "/MCU/STAT_LED") (pinfunction "PB2") (pintype "bidirectional"))
     (pad "15" smd rect (at 2 4.25 135) (size 1.6 0.55) (layers "F.Cu" "F.Paste" "F.Mask")
       (net 69 "/MCU/SDO") (pinfunction "PB3") (pintype "bidirectional"))
@@
   )
   (footprint "Button_Switch_THT:SW_PUSH_6mm_H5mm" (layer "B.Cu")
-    (at 115.6625 81.75 180)
+    (at 110.4125 81.75 180)
     (descr "tactile push button, 6x6mm e.g. PHAP33xx series, height=5mm")
     (tags "tact sw push 6mm")
@@
   (segment (start 208.775 77.775) (end 209 78) (width 0.45) (layer "F.Cu") (net 1))
   (segment (start 215.83 82.33) (end 215.83 81.85) (width 0.3) (layer "F.Cu") (net 1))
+  (segment (start 131.55 77.05) (end 132.25 77.75) (width 0.6) (layer "F.Cu") (net 1))
   (segment (start 204.225 76.4) (end 204.225 77.775) (width 0.45) (layer "F.Cu") (net 1))
   (segment (start 206.175 83.6) (end 206.175 82.325) (width 0.45) (layer "F.Cu") (net 1))
@@
   (segment (start 208.775 76.4) (end 208.775 77.775) (width 0.45) (layer "F.Cu") (net 1))
   (segment (start 206.175 82.325) (end 206.5 82) (width 0.45) (layer "F.Cu") (net 1))
+  (segment (start 130.9375 77.05) (end 131.55 77.05) (width 0.6) (layer "F.Cu") (net 1))
+  (via (at 132.25 77.75) (size 0.8) (drill 0.4) (layers "F.Cu" "B.Cu") (net 1))
   (segment (start 204.3 87.2) (end 204.3 85.75) (width 1) (layer "F.Cu") (net 3))
+  (segment (start 133.5625 76.95) (end 135.95 76.95) (width 0.6) (layer "F.Cu") (net 3))
   (segment (start 148.749963 82.578464) (end 148.421536 82.578464) (width 0.55) (layer "F.Cu") (net 3))
   (segment (start 190.5 69.3125) (end 193 69.3125) (width 1) (layer "F.Cu") (net 3))
@@
   (segment (start 203.55 93.45) (end 201.95 93.45) (width 1) (layer "F.Cu") (net 3))
   (segment (start 207.475 74.925) (end 206.55 74) (width 0.45) (layer "F.Cu") (net 3))
+  (segment (start 135.95 76.95) (end 136.5 77.5) (width 0.6) (layer "F.Cu") (net 3))
   (segment (start 203.6 89.5) (end 203.6 87.9) (width 1) (layer "F.Cu") (net 3))
   (via (at 145.5 84) (size 0.8) (drill 0.4) (layers "F.Cu" "B.Cu") (net 3))
+  (via (at 136.5 77.5) (size 0.8) (drill 0.4) (layers "F.Cu" "B.Cu") (net 3))
   (via (at 201.95 93.45) (size 0.8) (drill 0.4) (layers "F.Cu" "B.Cu") (net 3))
+  (segment (start 145.5 84) (end 138.5 84) (width 1) (layer "B.Cu") (net 3))
+  (segment (start 95.5 77.75) (end 95.5 69.5) (width 1) (layer "B.Cu") (net 3))
   (segment (start 185.5 88) (end 167.5 88) (width 1) (layer "B.Cu") (net 3))
+  (segment (start 99.5 86.25) (end 101.75 84) (width 0.25) (layer "B.Cu") (net 3))
+  (segment (start 110.4125 86.25) (end 112.6625 84) (width 0.25) (layer "B.Cu") (net 3))
+  (segment (start 101.75 84) (end 95.5 77.75) (width 1) (layer "B.Cu") (net 3))
   (segment (start 201.95 93.45) (end 196.5 88) (width 1) (layer "B.Cu") (net 3))
   (segment (start 152 91) (end 145.5 84.5) (width 1) (layer "B.Cu") (net 3))
   (segment (start 145.5 84.5) (end 145.5 84) (width 1) (layer "B.Cu") (net 3))
+  (segment (start 138.5 84) (end 113.25 84) (width 1) (layer "B.Cu") (net 3))
   (segment (start 167.5 88) (end 164.5 91) (width 1) (layer "B.Cu") (net 3))
+  (segment (start 103.9125 86.25) (end 106.1625 84) (width 0.25) (layer "B.Cu") (net 3))
+  (segment (start 106.75 84) (end 101.75 84) (width 1) (layer "B.Cu") (net 3))
+  (segment (start 94.75 86.25) (end 99.5 86.25) (width 0.25) (layer "B.Cu") (net 3))
   (segment (start 180.16 92.65) (end 181.35 92.65) (width 1) (layer "B.Cu") (net 3))
   (segment (start 164.5 91) (end 152 91) (width 1) (layer "B.Cu") (net 3))
+  (segment (start 106.1625 84) (end 106.75 84) (width 0.25) (layer "B.Cu") (net 3))
+  (segment (start 88.25 86.25) (end 94.75 86.25) (width 0.25) (layer "B.Cu") (net 3))
   (segment (start 181.35 92.65) (end 186 88) (width 1) (layer "B.Cu") (net 3))
+  (segment (start 136.5 77.5) (end 136.5 82) (width 0.6) (layer "B.Cu") (net 3))
   (segment (start 196.5 88) (end 185.5 88) (width 1) (layer "B.Cu") (net 3))
+  (segment (start 136.5 82) (end 138.5 84) (width 0.6) (layer "B.Cu") (net 3))
+  (segment (start 113.25 84) (end 106.75 84) (width 1) (layer "B.Cu") (net 3))
+  (segment (start 112.6625 84) (end 113.25 84) (width 0.25) (layer "B.Cu") (net 3))
   (segment (start 142.5 90) (end 142.5 91.156498) (width 0.55) (layer "F.Cu") (net 4))
   (segment (start 141.328249 92.328249) (end 141.171751 92.328249) (width 0.55) (layer "F.Cu") (net 4))
@@
   (segment (start 133.505204 89.494796) (end 132.994796 89.494796) (width 0.55) (layer "F.Cu") (net 5))
   (segment (start 140.828427 90.5) (end 139 90.5) (width 0.55) (layer "F.Cu") (net 5))
+  (via (at 106.3375 82.5) (size 0.8) (drill 0.4) (layers "F.Cu" "B.Cu") (net 20))
+  (segment (start 103.9125 81.75) (end 105.5875 81.75) (width 0.25) (layer "B.Cu") (net 20))
+  (segment (start 107.0875 81.75) (end 106.3375 82.5) (width 0.25) (layer "B.Cu") (net 20))
+  (segment (start 110.4125 81.75) (end 107.0875 81.75) (width 0.25) (layer "B.Cu") (net 20))
+  (segment (start 105.5875 81.75) (end 106.3375 82.5) (width 0.25) (layer "B.Cu") (net 20))
+  (via (at 90.6875 84.25) (size 0.8) (drill 0.4) (layers "F.Cu" "B.Cu") (net 21))
+  (segment (start 90.6875 84.25) (end 90.6875 84.1875) (width 0.25) (layer "B.Cu") (net 21))
+  (segment (start 93.1875 81.75) (end 90.6875 84.25) (width 0.25) (layer "B.Cu") (net 21))
+  (segment (start 94.75 81.75) (end 93.1875 81.75) (width 0.25) (layer "B.Cu") (net 21))
+  (segment (start 90.6875 84.1875) (end 88.25 81.75) (width 0.25) (layer "B.Cu") (net 21))
   (segment (start 189.5 96) (end 191.5 96) (width 1) (layer "F.Cu") (net 24))
+  (segment (start 142.209798 76.75) (end 140.25 76.75) (width 0.55) (layer "F.Cu") (net 24))
+  (segment (start 138 79) (end 135 79) (width 0.55) (layer "F.Cu") (net 24))
+  (segment (start 143.974695 78.514897) (end 142.209798 76.75) (width 0.55) (layer "F.Cu") (net 24))
   (segment (start 192.31 95.19) (end 192.86 95.19) (width 1) (layer "F.Cu") (net 24))
+  (segment (start 140.25 76.75) (end 138 79) (width 0.55) (layer "F.Cu") (net 24))
   (segment (start 191.5 96) (end 192.31 95.19) (width 1) (layer "F.Cu") (net 24))
   (segment (start 174.25 92.81) (end 174.25 94.25) (width 1.6) (layer "F.Cu") (net 25))
@@
   (segment (start 192.5 79.5) (end 190.5 77.5) (width 0.45) (layer "F.Cu") (net 50))
   (segment (start 204.661524 79.5) (end 192.5 79.5) (width 0.45) (layer "F.Cu") (net 50))
+  (segment (start 137.5 72.5) (end 137.5 69.5) (width 1) (layer "F.Cu") (net 67))
+  (segment (start 138 74.0875) (end 138 73) (width 1) (layer "F.Cu") (net 67))
+  (segment (start 138 73) (end 137.5 72.5) (width 1) (layer "F.Cu") (net 67))
   (segment (start 152 86.6445) (end 150.972927 86.6445) (width 0.55) (layer "F.Cu") (net 69))
   (segment (start 160.135 87.04) (end 160.46 87.04) (width 0.55) (layer "F.Cu") (net 69))
@@
   (segment (start 151.229798 85.77) (end 149.985103 84.525305) (width 0.55) (layer "F.Cu") (net 70))
   (segment (start 158.865 85.77) (end 151.229798 85.77) (width 0.55) (layer "F.Cu") (net 70))
+  (segment (start 133.125 78.95) (end 133.175 79) (width 0.6) (layer "F.Cu") (net 73))
+  (segment (start 130.9375 78.95) (end 133.125 78.95) (width 0.6) (layer "F.Cu") (net 73))
+  (segment (start 129.5875 76.1625) (end 129.5875 75) (width 0.6) (layer "F.Cu") (net 74))
+  (segment (start 129.0625 76.6875) (end 129.5875 76.1625) (width 0.6) (layer "F.Cu") (net 74))
+  (segment (start 129.0625 78) (end 129.0625 76.6875) (width 0.6) (layer "F.Cu") (net 74))
+  (segment (start 131.4625 75.05) (end 131.4125 75) (width 0.6) (layer "F.Cu") (net 75))
+  (segment (start 133.5625 75.05) (end 131.4625 75.05) (width 0.6) (layer "F.Cu") (net 75))
+  (segment (start 137.9125 76) (end 138 75.9125) (width 0.6) (layer "F.Cu") (net 76))
+  (segment (start 135.4375 76) (end 137.9125 76) (width 0.6) (layer "F.Cu") (net 76))
   (segment (start 219 78.5) (end 219 83) (width 0.3) (layer "F.Cu") (net 78))
   (segment (start 220 84) (end 220 85.0875) (width 0.3) (layer "F.Cu") (net 78))

Commit message: Do more
Routing:
- net /EN: track 14.3 -> 75.0 mm, vias 0 -> 2
- net /STEP: track 0.00 -> 57.2 mm, vias 0 -> 2
- net /DIR: track 0.00 -> 55.4 mm, vias 0 -> 2
- net /MCU/TXD: track 0.00 -> 51.3 mm, vias 0 -> 2
- net /MCU/RXD: track 0.00 -> 48.5 mm, vias 0 -> 1
- net /MCU/TFT_A0: track 0.00 -> 44.0 mm, vias 0 -> 2
- net Net-(C404-Pad2): track 0.00 -> 43.5 mm
- net /MCU/TFT_CS: track 0.00 -> 43.4 mm, vias 0 -> 2
- net /MCU/RST: track 0.00 -> 37.6 mm
- net /MCU/TFT_RESET: track 0.00 -> 32.4 mm
- net Net-(R202-Pad1): track 0.00 -> 31.8 mm, vias 0 -> 2
- net Net-(R201-Pad1): track 0.00 -> 30.1 mm, vias 0 -> 2
- net +5V: track 226.6 -> 245.0 mm, vias 3 -> 5
- net Net-(J402-Pad4): track 0.00 -> 13.8 mm
- net /MCU/SCK: track 0.00 -> 11.1 mm
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
Commit message: Add new connector
Parts:
- removed D101: 1.8TFT, Connector_JST:JST_EH_B8B-EH-A_1x08_P2.50mm_Vertical
- added C102: EYE_SP, Connector_FFC-FPC:Hirose_FH12-18S-0.5SH_1x18-1MP_P0.50mm_Horizontal, F.Cu at (124.0, 72.0)
- added TP103: TestPoint, TestPoint:TestPoint_Pad_1.0x1.0mm, F.Cu at (120.5, 79.0)
- added TP104: TestPoint, TestPoint:TestPoint_Pad_1.0x1.0mm, F.Cu at (120.5, 81.0)
- added TP105: TestPoint, TestPoint:TestPoint_Pad_1.0x1.0mm, F.Cu at (120.5, 83.0)
- added TP106: TestPoint, TestPoint:TestPoint_Pad_1.0x1.0mm, F.Cu at (120.5, 85.0)
- added TP107: TestPoint, TestPoint:TestPoint_Pad_1.0x1.0mm, F.Cu at (131.0, 85.2)
- added TP108: TestPoint, TestPoint:TestPoint_Pad_1.0x1.0mm, F.Cu at (127.0, 85.0)
- moved Q101 7.56 mm to (137.5, 77.0), turned to -90 degrees
- moved R101 7.51 mm to (138.5, 72.9), turned to -90 degrees
- moved R103 6.94 mm to (134.5, 69.0), turned to 180 degrees
- moved R102 4.28 mm to (134.5, 76.5), turned to 90 degrees
- moved Q102 3.63 mm to (135.5, 72.5), turned to 90 degrees
Connections:
- net /MCU/SCK renamed /SCK
- net /MCU/SDI renamed /SDI
- net /MCU/SDO renamed /SDO
- U201 pad 10: /MCU/TFT_A0 -> /SD_CS
- U201 pad 11: unconnected-(U201-Pad11) -> /DATA/COMMAND
- U201 pad 2: /MCU/TFT_RESET -> /RESET
- U201 pad 9: /MCU/TFT_CS -> /TFT_CS
Routing:
- net /DATA/COMMAND: track 0.00 -> 48.1 mm, vias 0 -> 2
- net /MCU/TFT_A0: track 44.0 -> 0.00 mm, vias 2 -> 0
- net /TFT_CS: track 0.00 -> 43.6 mm, vias 0 -> 2
- net /MCU/TFT_CS: track 43.4 -> 0.00 mm, vias 2 -> 0
- net /SD_CS: track 0.00 -> 40.5 mm, vias 0 -> 2
- net /MCU/TFT_RESET: track 32.4 -> 0.00 mm
- net /RESET: track 0.00 -> 31.9 mm
- net +5V: track 245.0 -> 261.0 mm, vias 5 -> 6
- net /TFT_LED: track 4.79 -> 17.9 mm
- net /SDO: track 14.8 -> 24.7 mm
- net /SDI: track 9.40 -> 18.4 mm, vias 0 -> 1
- net /SCK: track 11.1 -> 17.7 mm, vias 0 -> 1
- net GND: track 22.9 -> 24.7 mm, vias 26 -> 27
- net /EN: track 75.0 -> 73.7 mm

Commit message: Route all
Parts:
- moved TP107 5.71 mm to (126.0, 88.0)
- moved SW201 3.04 mm to (150.8, 96.8)
Routing:
- net /MCU/STOP/MODE: track 8.61 -> 79.1 mm, vias 1 -> 3
- net /MCU/AnalogP: track 0.00 -> 65.0 mm, vias 0 -> 2
- net /SCK: track 17.7 -> 81.5 mm, vias 1 -> 2
- net /EncB: track 0.00 -> 59.2 mm, vias 0 -> 2
- net /MCU/START: track 7.12 -> 66.2 mm, vias 1 -> 3
- net /EncA: track 0.00 -> 56.8 mm, vias 0 -> 2
- net /SDI: track 18.4 -> 74.2 mm, vias 1 -> 0
- net /SDO: track 24.7 -> 76.3 mm
- net /MCU/AnalogI: track 0.00 -> 50.8 mm, vias 0 -> 1
- net /MCU/AnalogD: track 0.00 -> 38.3 mm, vias 0 -> 1
- net +5V: track 261.0 -> 297.9 mm
- net /MCU/RST: track 37.6 -> 63.3 mm, vias 0 -> 2
- net /MCU/STAT_LED: track 0.00 -> 23.5 mm, vias 0 -> 2
- net GND: track 24.7 -> 41.3 mm, vias 27 -> 32
- net Net-(D201-Pad1): track 0.00 -> 7.13 mm
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