File: Hardware/PendulumController/PendulumController.kicad_pcb (KiCad board)
At the start: 2 copper layers, 157 x 47 mm, 83 parts, among them J101 MOTOR, J102 ENCODER, J201 ICSP, J202 Limit, J302 19V Input, J401 USBC, J402 PROG, Q101 MMBT3904, Q102 MMBT3906, SW201 RESET, SW202 START_SW, SW203 STOP/MODE_SW, U201 ATmega328P, U301 NCV1117ST50T3G, U401 FT232RL, Y201 16mHz

Commit message: more work
Routing:
- net Net-(R202-Pad1): track 13.8 -> 65.7 mm, vias 1 -> 2
- net Net-(R201-Pad1): track 13.5 -> 61.9 mm, vias 1 -> 2
- net Net-(C404-Pad2): track 0.00 -> 40.9 mm, vias 0 -> 2
- net /SD_CS: track 22.6 -> 48.4 mm, vias 1 -> 2
- net /DATA/COMMAND: track 34.6 -> 9.99 mm, vias 1 -> 0
- net /SDI: track 14.5 -> 36.0 mm, vias 1 -> 2
- net /TFT_CS: track 32.3 -> 11.0 mm, vias 1 -> 0
- net GND: track 39.6 -> 41.3 mm, vias 27 -> 28
