File: Hardware/PendulumController/PendulumController.kicad_sch (KiCad schematic)
At the start: 19 parts, among them J101 MOTOR, J102 ENCODER, Q101 MMBT3904, Q102 MMBT3906

Commit message: Add new connector
Parts:
- removed D101: 1.8TFT, Connector_JST:JST_EH_B8B-EH-A_1x08_P2.50mm_Vertical, symbol KenwoodFox:1.8TFT
- added C102: EYE_SP, Connector_FFC-FPC:Hirose_FH12-18S-0.5SH_1x18-1MP_P0.50mm_Horizontal, symbol KenwoodFox:EYE_SP
- added TP103, TP104, TP105, TP106, TP107, TP108: TestPoint, TestPoint:TestPoint_Pad_1.0x1.0mm, symbol Connector:TestPoint
Connections:
- net +5V: now also C102.18 (VCC)
- net GND: now also C102.16 (GND)
- net TFT_LED: now also C102.17 (BackLite)
- new net DATA/COMMAND: C102.12 (D/C), TP106.1
- new net RESET: C102.11 (RESET), TP107.1
- new net SCK: C102.15 (SCK), TP103.1
- new net SDI: C102.14 (SDO), TP104.1
- new net SDO: C102.13 (SDI), TP105.1
- new net SD_CS: C102.9 (SD_CS)
- new net TFT_CS: C102.10 (DISP_CS), TP108.1
- no-connect marks 4 -> 12
Other:
- sheet MCU ports: added SDI, SD_CS, TFT_DC; removed TFT_A0
- moved on the sheet: Q101, Q102, R101, R102, R103

Commit message: Fix ERC
Changed lines of the file:
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@@
   (junction (at 260.985 36.195) (diameter 0) (color 0 0 0 0)
+  )
+  (junction (at 151.13 182.245) (diameter 0) (color 0 0 0 0)
   )
   (junction (at 233.68 91.44) (diameter 0) (color 0 0 0 0)
@@
     (stroke (width 0) (type default) (color 0 0 0 0))
   )
+  (wire (pts (xy 151.13 182.245) (xy 160.02 182.245))
+    (stroke (width 0) (type default) (color 0 0 0 0))
+  )
   (wire (pts (xy 226.695 91.44) (xy 233.68 91.44))
     (stroke (width 0) (type default) (color 0 0 0 0))
@@
     (stroke (width 0) (type default) (color 0 0 0 0))
   )
-  (wire (pts (xy 149.86 182.245) (xy 160.02 182.245))
+  (wire (pts (xy 149.86 182.245) (xy 151.13 182.245))
     (stroke (width 0) (type default) (color 0 0 0 0))
   )
@@
     )
   )
-  (symbol (lib_id "power:GND") (at 254.635 116.84 0) (unit 1)
+  (symbol (lib_name "GND_2") (lib_id "power:GND") (at 254.635 116.84 0) (unit 1)
     (in_bom yes) (on_board yes)
     (property "Reference" "#PWR0104" (id 0) (at 254.635 123.19 0)
@@
     )
   )
-  (symbol (lib_id "power:GND") (at 249.555 116.84 0) (unit 1)
+  (symbol (lib_name "GND_3") (lib_id "power:GND") (at 249.555 116.84 0) (unit 1)
     (in_bom yes) (on_board yes)
     (property "Reference" "#PWR0103" (id 0) (at 249.555 123.19 0)
@@
     (pin "1")
   )
-  (symbol (lib_id "power:+5V") (at 249.555 75.565 0) (unit 1)
+  (symbol (lib_name "+5V_1") (lib_id "power:+5V") (at 249.555 75.565 0) (unit 1)
     (in_bom yes) (on_board yes)
     (property "Reference" "#PWR0106" (id 0) (at 249.555 79.375 0)
@@
     (pin "1")
   )
-  (symbol (lib_id "power:GND") (at 127 189.865 0) (unit 1)
+  (symbol (lib_name "GND_5") (lib_id "power:GND") (at 127 189.865 0) (unit 1)
     (in_bom yes) (on_board yes)
     (property "Reference" "#PWR0142" (id 0) (at 127 196.215 0)
@@
     (pin "2")
   )
-  (symbol (lib_id "power:GND") (at 132.715 123.825 0) (unit 1)
+  (symbol (lib_name "GND_4") (lib_id "power:GND") (at 132.715 123.825 0) (unit 1)
     (in_bom yes) (on_board yes)
     (property "Reference" "#PWR0139" (id 0) (at 132.715 130.175 0)
@@
     (pin "1")
   )
-  (symbol (lib_id "power:+5V") (at 268.605 29.21 0) (unit 1)
+  (symbol (lib_id "power:PWR_FLAG") (at 151.13 182.245 0) (unit 1)
+    (in_bom yes) (on_board yes) (fields_autoplaced)
+    (property "Reference" "#FLG0104" (id 0) (at 151.13 180.34 0)
+      (effects (font (size 1.27 1.27)) hide)
+    )
+    (property "Value" "PWR_FLAG" (id 1) (at 151.13 176.53 0)
+      (effects (font (size 1.27 1.27)) hide)
+    )
+    (property "Footprint" "" (id 2) (at 151.13 182.245 0)
+      (effects (font (size 1.27 1.27)) hide)
+    )
+    (property "Datasheet" "~" (id 3) (at 151.13 182.245 0)
+      (effects (font (size 1.27 1.27)) hide)
+    )
+    (pin "1")
+  )
+  (symbol (lib_name "+5V_3") (lib_id "power:+5V") (at 268.605 29.21 0) (unit 1)
     (in_bom yes) (on_board yes)
     (property "Reference" "#PWR0132" (id 0) (at 268.605 33.02 0)
@@
     (pin "2")
   )
-  (symbol (lib_id "power:+5V") (at 142.875 168.91 0) (unit 1)
+  (symbol (lib_name "+5V_2") (lib_id "power:+5V") (at 142.875 168.91 0) (unit 1)
     (in_bom yes) (on_board yes)
     (property "Reference" "#PWR0143" (id 0) (at 142.875 172.72 0)
@@
     (pin "3")
   )
-  (symbol (lib_id "power:GND") (at 265.43 85.725 0) (unit 1)
+  (symbol (lib_name "GND_1") (lib_id "power:GND") (at 265.43 85.725 0) (unit 1)
     (in_bom yes) (on_board yes)
     (property "Reference" "#PWR0105" (id 0) (at 265.43 92.075 0)
@@
       (reference "#FLG0103") (unit 1) (value "PWR_FLAG") (footprint "")
     )
+    (path "/c63be524-fd1c-4261-9a24-8b77af34c624"
+      (reference "#FLG0104") (unit 1) (value "PWR_FLAG") (footprint "")
+    )
     (path "/2ecf2374-9c1c-4e92-a809-f5005df04ae1"

Commit message: Last cleanups!
Parts:
- removed R103: TBD, Resistor_SMD:R_0805_2012Metric, symbol Device:R_Small
Connections:
- net EN: now also A101.9 (~{ENABLE}); no longer A101.14 (~{SLEEP}), JP101.2 (B)
- net TFT_LED: now also Q102.3 (C)
- new net: A101.14 (~{SLEEP}), JP101.2 (B)
- no-connect marks 12 -> 11
Changed lines of the file:
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@@
   (junction (at 151.13 182.245) (diameter 0) (color 0 0 0 0)
-  )
-  (junction (at 233.68 91.44) (diameter 0) (color 0 0 0 0)
   )
   (junction (at 260.985 33.655) (diameter 0) (color 0 0 0 0)
@@
   (no_connect (at 239.395 103.505))
   (no_connect (at 120.015 114.935))
-  (no_connect (at 239.395 93.345))
   (no_connect (at 120.015 109.855))
   (no_connect (at 239.395 108.585))
@@
     (stroke (width 0) (type default) (color 0 0 0 0))
   )
+  (wire (pts (xy 226.695 93.345) (xy 239.395 93.345))
+    (stroke (width 0) (type default) (color 0 0 0 0))
+  )
   (wire (pts (xy 101.6 94.615) (xy 120.015 94.615))
     (stroke (width 0) (type default) (color 0 0 0 0))
@@
     (stroke (width 0) (type default) (color 0 0 0 0))
   )
-  (wire (pts (xy 142.875 182.245) (xy 144.78 182.245))
-    (stroke (width 0) (type default) (color 0 0 0 0))
-  )
   (wire (pts (xy 130.175 73.025) (xy 130.175 75.565))
     (stroke (width 0) (type default) (color 0 0 0 0))
@@
     (stroke (width 0) (type default) (color 0 0 0 0))
   )
-  (wire (pts (xy 226.695 91.44) (xy 233.68 91.44))
-    (stroke (width 0) (type default) (color 0 0 0 0))
-  )
   (wire (pts (xy 101.6 89.535) (xy 120.015 89.535))
     (stroke (width 0) (type default) (color 0 0 0 0))
@@
     (stroke (width 0) (type default) (color 0 0 0 0))
   )
-  (wire (pts (xy 149.86 182.245) (xy 151.13 182.245))
+  (wire (pts (xy 142.875 182.245) (xy 151.13 182.245))
     (stroke (width 0) (type default) (color 0 0 0 0))
   )
@@
     (effects (font (size 1.27 1.27)) (justify left bottom))
   )
+  (label "EN" (at 226.695 93.345 0)
+    (effects (font (size 1.27 1.27)) (justify left bottom))
+  )
   (label "SDI" (at 101.6 84.455 0)
     (effects (font (size 1.27 1.27)) (justify left bottom))
@@
   (label "EN" (at 85.725 76.2 180)
     (effects (font (size 1.27 1.27)) (justify right bottom))
-  )
-  (label "EN" (at 226.695 91.44 0)
-    (effects (font (size 1.27 1.27)) (justify left bottom))
   )
   (label "SDI" (at 162.56 78.74 0)
@@
     (pin "1")
   )
-  (symbol (lib_id "Device:R_Small") (at 147.32 182.245 90) (unit 1)
-    (in_bom yes) (on_board yes)
-    (property "Reference" "R103" (id 0) (at 144.145 184.15 90))
-    (property "Value" "TBD" (id 1) (at 145.415 186.055 90))
-    (property "Footprint" "Resistor_SMD:R_0805_2012Metric" (id 2) (at 147.32 182.245 0)
-      (effects (font (size 1.27 1.27)) hide)
-    )
-    (property "Datasheet" "~" (id 3) (at 147.32 182.245 0)
-      (effects (font (size 1.27 1.27)) hide)
-    )
-    (pin "1")
-    (pin "2")
-  )
   (symbol (lib_id "Mechanical:MountingHole") (at 14.605 194.945 0) (unit 1)
     (in_bom yes) (on_board yes) (fields_autoplaced)
@@
       (reference "R102") (unit 1) (value "TBD") (footprint "Resistor_SMD:R_0805_2012Metric")
     )
-    (path "/754991e1-0f30-4549-aa1e-b6eb10f1a13f"
-      (reference "R103") (unit 1) (value "TBD") (footprint "Resistor_SMD:R_0805_2012Metric")
-    )
     (path "/4c5d1f0c-71b8-4a0e-888c-794bf6e4c7a4/888b06ea-8071-472f-8dff-86516940ac0d"
